File: SMSSchematic.sch (KiCad schematic (older format))
At the start: 21 parts, among them CN6 JOYSTICK2, CN7 JOYSTICK1, IC1 CXK3864, IC2 4168, IC3 315-5124, IC4 4168, IC5 4168, SW2 PAUSE, U2 Z80, U3 315-5216

Commit message: Cartridge and card slots
Parts:
- added CN2: SMS_Card_Port, Socket_Strips:Socket_Strip_Angled_2x17, symbol SMS_Card_Port
- added CN3: SMS_Cartridge, SMSFootprints:EDGE_CONN_50P_0p1pitch, symbol SMS_Cartridge
- added CN4: SMS_Cartridge, SMSFootprints:SMS_CartridgeEdgeConn, symbol SMS_Cartridge
- R4: footprint (none) -> Resistors_ThroughHole:Resistor_Horizontal_RM10mm
- SW2: footprint (none) -> Buttons_Switches_ThroughHole:SW_PUSH_SMALL
Connections:
- net A0: now also CN2.25 (A0), CN3.25 (A0), CN4.25 (A0)
- net A1: now also CN2.26 (A1), CN3.26 (A1), CN4.26 (A1)
- net A10: now also CN2.12 (A10), CN3.12 (A10), CN4.12 (A10)
- net A11: now also CN2.10 (A11), CN3.10 (A11), CN4.10 (A11)
- net A12: now also CN2.33 (A12), CN3.33 (A12), CN4.33 (A12)
- net A13: now also CN2.7 (A13), CN3.7 (A13), CN4.7 (A13)
- net A14: now also CN2.6 (A14), CN3.6 (A14), CN4.6 (A14)
- net A2: now also CN2.27 (A2), CN3.27 (A2), CN4.27 (A2)
- net A3: now also CN2.28 (A3), CN3.28 (A3), CN4.28 (A3)
- net A4: now also CN2.29 (A4), CN3.29 (A4), CN4.29 (A4)
- net A5: now also CN2.30 (A5), CN3.30 (A5), CN4.30 (A5)
- net A6: now also CN2.31 (A6), CN3.31 (A6), CN4.31 (A6)
- net A7: now also CN2.32 (A7), CN3.32 (A7), CN4.32 (A7)
- net A8: now also CN2.8 (A8), CN3.8 (A8), CN4.8 (A8)
- net A9: now also CN2.9 (A9), CN3.9 (A9), CN4.9 (A9)
- net D0: now also CN2.24 (D0), CN3.24 (D0), CN4.24 (D0)
- net D1: now also CN2.23 (D1), CN3.23 (D1), CN4.23 (D1)
- net D2: now also CN2.22 (D2), CN3.22 (D2), CN4.22 (D2)
- net D3: now also CN2.18 (D3), CN3.18 (D3), CN4.18 (D3)
- net D4: now also CN2.17 (D4), CN3.17 (D4), CN4.17 (D4)
- net D5: now also CN2.16 (D5), CN3.16 (D5), CN4.16 (D5)
- net D6: now also CN2.15 (D6), CN3.15 (D6), CN4.15 (D6)
- net D7: now also CN2.14 (D7), CN3.14 (D7), CN4.14 (D7)
- net GNDPWR: now also CN2.19 (GND), CN2.20 (GND), CN2.21 (GND), CN3.19 (GND), CN3.20 (GND), CN3.21 (GND), CN4.19 (GND), CN4.20 (GND), CN4.21 (GND)
- net VCC: now also CN2.1 (+5V), CN2.35 (+5V), CN3.1 (+5V), CN3.35 (+5V), CN4.1 (+5V), CN4.35 (+5V)
- new net: CN2.11 (EXM2), CN3.11 (EXM2), CN4.11 (EXM2)
- new net: CN2.2 (WR), CN3.2 (WR), CN4.2 (WR)
- new net: CN2.3 (MReq), CN3.3 (MReq), CN4.3 (MReq)
- new net: CN2.34 (CONT), CN3.34 (CONT), CN4.34 (CONT)
- new net: CN2.4 (RD), CN3.4 (RD), CN4.4 (RD)
- new net: CN2.5 (EXM1), CN3.5 (EXM1), CN4.5 (EXM1)
- new net: CN3.36 (A15), CN4.36 (A15)
- new net: CN3.37 (M1), CN4.37 (M1)
- new net: CN3.38 (IOReq), CN4.38 (IOReq)
- new net: CN3.39 (Refresh), CN4.39 (Refresh)
- new net: CN3.40 (Halt), CN4.40 (Halt)
- new net: CN3.41 (Wait), CN4.41 (Wait)
- new net: CN3.42 (Int), CN4.42 (Int)
- new net: CN3.43 (KILLGA), CN4.43 (KILLGA)
- new net: CN3.44 (BusReq), CN4.44 (BusReq)
- new net: CN3.45 (BusAck), CN4.45 (BusAck)
- new net: CN3.46 (Reset), CN4.46 (Reset)
- new net: CN3.47 (Clock), CN4.47 (Clock)
- new net: CN3.48 (KBSEL), CN4.48 (KBSEL)
- new net: CN3.49 (CSRAM), CN4.49 (CSRAM)
- new net: CN3.50 (NMI), CN4.50 (NMI)

Commit message: Cartridge, Card and Gameport slots in place
Parts:
- CN3: value SMS_Cartridge -> CartridgeSlot
- CN4: value SMS_Cartridge -> EdgeConnector
Connections:
- net 1DN: now also U3.26 (1DN)
- net 1LE: now also U3.27 (1LE)
- net 1RI: now also U3.28 (1RI)
- net 1TH: now also U3.31 (1TH)
- net 1TL: now also U3.29 (1TL)
- net 1TR: now also U3.30 (1TR)
- net 1UP: now also U3.25 (1UP)
- net 2DN: now also U3.39 (2DN)
- net 2LE: now also U3.38 (2LE)
- net 2RI: now also U3.37 (2RI)
- net 2TH: now also U3.34 (2TH)
- net 2TL: now also U3.36 (2TL)
- net 2TR: now also U3.35 (2TR)
- net 2UP: now also U3.40 (2UP)
- net CE2: now also CN2.13 (CE)
- net CE3: now also CN3.13 (CE)
- net CE4: now also CN4.13 (CE)
- net MREQ: now also CN2.3 (MReq), CN3.3 (MReq), CN4.3 (MReq)
- net RD: now also CN2.4 (RD), CN3.4 (RD), CN4.4 (RD)
- net WR: now also CN2.2 (WR), CN3.2 (WR), CN4.2 (WR)
- net EXM2: now reaches CN2.11 (EXM2), CN3.11 (EXM2), CN4.11 (EXM2)
- net EXM1: now reaches CN2.5 (EXM1), CN3.5 (EXM1), CN4.5 (EXM1)
- net at IC3.36 (#WE1), IC5.27 (#WE): no longer IC3.37 (#WE0), IC4.27 (#WE)
- new net: IC3.37 (#WE0), IC4.27 (#WE)
- no-connect marks 2 -> 3

Commit message: Beginnings of video generation and clocking
Parts:
- renumbered U3 to IC4
Connections:
- net at IC4.24 (#CSRAM): no longer IC3.15 (#CSRAM)
- net at IC4.33 (#H-L): no longer IC3.35 (#H-L)
- net Video Encoder/AUDIO: now reaches IC3.19 (AUDIO)
- net Video Encoder/R: now reaches IC3.26 (R)
- net Video Encoder/G: now reaches IC3.27 (G)
- net Video Encoder/B: now reaches IC3.28 (B)
- net Video Encoder/CSYNC: now reaches IC3.29 (#CSYNC)
- net VDP_CLK: now reaches IC3.30 (XTAL1)
- net Video Encoder/NTSC/PAL: now reaches IC3.57 (PAL/#NTSC)
- no-connect marks 3 -> 6
Changed lines of the file:
@@
 LIBS:contrib
 LIBS:valves
+LIBS:SMS_Chips
 LIBS:SMSSchematic-cache
 EELAYER 25 0
@@
 $Descr A3 16535 11693
 encoding utf-8
-Sheet 1 2
+Sheet 1 4
 Title "Power Base"
 Date ""
@@
 $EndComp
 $Comp
-L VCC #PWR01
+L VCC #PWR21
 U 1 1 56960B2F
 P 14450 950
-F 0 "#PWR01" H 14450 800 50  0001 C CNN
+F 0 "#PWR21" H 14450 800 50  0001 C CNN
 F 1 "VCC" H 14450 1100 50  0000 C CNN
 F 2 "" H 14450 950 50  0000 C CNN
@@
 $EndComp
 $Comp
-L GNDPWR #PWR02
+L GNDPWR #PWR19
 U 1 1 56960B4E
 P 14150 1950
-F 0 "#PWR02" H 14150 1750 50  0001 C CNN
+F 0 "#PWR19" H 14150 1750 50  0001 C CNN
 F 1 "GNDPWR" H 14150 1820 50  0000 C CNN
 F 2 "" H 14150 1900 50  0000 C CNN
@@
 $EndComp
 $Comp
-L VCC #PWR03
+L VCC #PWR22
 U 1 1 56960E1C
 P 14450 2450
-F 0 "#PWR03" H 14450 2300 50  0001 C CNN
+F 0 "#PWR22" H 14450 2300 50  0001 C CNN
 F 1 "VCC" H 14450 2600 50  0000 C CNN
 F 2 "" H 14450 2450 50  0000 C CNN
@@
 $EndComp
 $Comp
-L GNDPWR #PWR04
+L GNDPWR #PWR20
 U 1 1 56960E22
 P 14150 3450
-F 0 "#PWR04" H 14150 3250 50  0001 C CNN
+F 0 "#PWR20" H 14150 3250 50  0001 C CNN
 F 1 "GNDPWR" H 14150 3320 50  0000 C CNN
 F 2 "" H 14150 3400 50  0000 C CNN
@@
 $EndComp
 $Comp
-L VCC #PWR05
+L VCC #PWR3
 U 1 1 5696703C
 P 1000 9600
-F 0 "#PWR05" H 1000 9450 50  0001 C CNN
+F 0 "#PWR3" H 1000 9450 50  0001 C CNN
 F 1 "VCC" H 1000 9750 50  0000 C CNN
 F 2 "" H 1000 9600 50  0000 C CNN
@@
 $EndComp
 $Comp
-L VCC #PWR06
+L VCC #PWR2
 U 1 1 569671B6
 P 800 9500
-F 0 "#PWR06" H 800 9350 50  0001 C CNN
+F 0 "#PWR2" H 800 9350 50  0001 C CNN
 F 1 "VCC" H 800 9650 50  0000 C CNN
 F 2 "" H 800 9500 50  0000 C CNN
@@
 $EndComp
 $Comp
-L GNDPWR #PWR07
+L GNDPWR #PWR6
 U 1 1 56967AD9
 P 3300 10500
-F 0 "#PWR07" H 3300 10300 50  0001 C CNN
+F 0 "#PWR6" H 3300 10300 50  0001 C CNN
 F 1 "GNDPWR" H 3300 10370 50  0000 C CNN
 F 2 "" H 3300 10450 50  0000 C CNN
@@
 $EndComp
 $Comp
-L VCC #PWR08
+L VCC #PWR5
 U 1 1 56967B0E
 P 3300 10000
-F 0 "#PWR08" H 3300 9850 50  0001 C CNN
+F 0 "#PWR5" H 3300 9850 50  0001 C CNN
 F 1 "VCC" H 3300 10150 50  0000 C CNN
 F 2 "" H 3300 10000 50  0000 C CNN
@@
 	3600 10300 3700 10400
 $Comp
-L VCC #PWR09
+L VCC #PWR7
 U 1 1 56967CC3
 P 3800 8800
-F 0 "#PWR09" H 3800 8650 50  0001 C CNN
+F 0 "#PWR7" H 3800 8650 50  0001 C CNN
 F 1 "VCC" H 3800 8950 50  0000 C CNN
 F 2 "" H 3800 8800 50  0000 C CNN
@@
 $EndComp
 $Comp
-L GNDPWR #PWR010
+L GNDPWR #PWR10
 U 1 1 56967E47
 P 5400 10500
-F 0 "#PWR010" H 5400 10300 50  0001 C CNN
+F 0 "#PWR10" H 5400 10300 50  0001 C CNN
 F 1 "GNDPWR" H 5400 10370 50  0000 C CNN
 F 2 "" H 5400 10450 50  0000 C CNN
@@
 $EndComp
 $Comp
-L VCC #PWR011
+L VCC #PWR9
 U 1 1 56967E76
 P 5400 10100
-F 0 "#PWR011" H 5400 9950 50  0001 C CNN
+F 0 "#PWR9" H 5400 9950 50  0001 C CNN
 F 1 "VCC" H 5400 10250 50  0000 C CNN
 F 2 "" H 5400 10100 50  0000 C CNN
@@
 $EndComp
 $Comp
-L GNDPWR #PWR012
+L GNDPWR #PWR13
 U 1 1 56968BC6
 P 7500 10500
-F 0 "#PWR012" H 7500 10300 50  0001 C CNN
+F 0 "#PWR13" H 7500 10300 50  0001 C CNN
 F 1 "GNDPWR" H 7500 10370 50  0000 C CNN
 F 2 "" H 7500 10450 50  0000 C CNN
@@
 $EndComp
 $Comp
-L VCC #PWR013
+L VCC #PWR12
 U 1 1 56968BCC
 P 7500 10100
-F 0 "#PWR013" H 7500 9950 50  0001 C CNN
+F 0 "#PWR12" H 7500 9950 50  0001 C CNN
 F 1 "VCC" H 7500 10250 50  0000 C CNN
 F 2 "" H 7500 10100 50  0000 C CNN
@@
 $EndComp
 $Comp
-L 315-5216 U3
+L 315-5216 IC4
 U 1 1 56969756
 P 9000 8900
-F 0 "U3" H 9000 8850 60  0000 C CNN
+F 0 "IC4" H 9000 8850 60  0000 C CNN
 F 1 "315-5216" H 9000 8950 60  0000 C CNN
 F 2 "SMSFootprints:DIP-42_W15.24mm" H 8700 8750 60  0001 C CNN
@@
 $EndComp
 $Comp
-L GNDPWR #PWR014
+L GNDPWR #PWR15
 U 1 1 569698AA
 P 9900 10500
-F 0 "#PWR014" H 9900 10300 50  0001 C CNN
+F 0 "#PWR15" H 9900 10300 50  0001 C CNN
 F 1 "GNDPWR" H 9900 10370 50  0000 C CNN
 F 2 "" H 9900 10450 50  0000 C CNN
@@
 $EndComp
 $Comp
-L VCC #PWR015
+L VCC #PWR14
 U 1 1 569698E5
 P 9900 10000
-F 0 "#PWR015" H 9900 9850 50  0001 C CNN
+F 0 "#PWR14" H 9900 9850 50  0001 C CNN
 F 1 "VCC" H 9900 10150 50  0000 C CNN
 F 2 "" H 9900 10000 50  0000 C CNN
@@
 $EndComp
 $Comp
-L GNDPWR #PWR016
+L GNDPWR #PWR17
 U 1 1 56970A1C
 P 13200 6700
-F 0 "#PWR016" H 13200 6500 50  0001 C CNN
+F 0 "#PWR17" H 13200 6500 50  0001 C CNN
 F 1 "GNDPWR" H 13200 6570 50  0000 C CNN
 F 2 "" H 13200 6650 50  0000 C CNN
@@
 $EndComp
 $Comp
-L VCC #PWR017
+L VCC #PWR16
 U 1 1 56970B70
 P 12400 6300
-F 0 "#PWR017" H 12400 6150 50  0001 C CNN
+F 0 "#PWR16" H 12400 6150 50  0001 C CNN
 F 1 "VCC" H 12400 6450 50  0000 C CNN
 F 2 "" H 12400 6300 50  0000 C CNN
@@
 	6700 7000 6800 7100
 $Comp
-L VCC #PWR018
+L VCC #PWR11
 U 1 1 56973A6B
 P 7500 9200
-F 0 "#PWR018" H 7500 9050 50  0001 C CNN
+F 0 "#PWR11" H 7500 9050 50  0001 C CNN
 F 1 "VCC" H 7500 9350 50  0000 C CNN
 F 2 "" H 7500 9200 50  0000 C CNN
@@
 IO\nGateArray\n
 $Comp
-L VCC #PWR019
+L VCC #PWR18
 U 1 1 56977967
 P 14000 7600
-F 0 "#PWR019" H 14000 7450 50  0001 C CNN
+F 0 "#PWR18" H 14000 7450 50  0001 C CNN
 F 1 "VCC" H 14000 7750 50  0000 C CNN
 F 2 "" H 14000 7600 50  0000 C CNN
@@
 $EndComp
 $Comp
-L VCC #PWR020
+L VCC #PWR23
 U 1 1 56977C2A
 P 15900 7600
-F 0 "#PWR020" H 15900 7450 50  0001 C CNN
+F 0 "#PWR23" H 15900 7450 50  0001 C CNN
 F 1 "VCC" H 15900 7750 50  0000 C CNN
 F 2 "" H 15900 7600 50  0000 C CNN
@@
 	3900 3400 4000 3300
 $Comp
-L GNDPWR #PWR?
+L GNDPWR #PWR4
 U 1 1 56973356
 P 2700 3500
-F 0 "#PWR?" H 2700 3300 50  0001 C CNN
+F 0 "#PWR4" H 2700 3300 50  0001 C CNN
 F 1 "GNDPWR" H 2700 3370 50  0000 C CNN
 F 2 "" H 2700 3450 50  0000 C CNN
@@
 $EndComp
 $Comp
-L VCC #PWR?
+L VCC #PWR1
 U 1 1 56973E46
 P 600 3000
-F 0 "#PWR?" H 600 2850 50  0001 C CNN
+F 0 "#PWR1" H 600 2850 50  0001 C CNN
 F 1 "VCC" H 600 3150 50  0000 C CNN
 F 2 "" H 600 3000 50  0000 C CNN
@@
 $EndComp
 $Comp
-L VCC #PWR?
+L VCC #PWR8
 U 1 1 56974234
 P 4400 3000
-F 0 "#PWR?" H 4400 2850 50  0001 C CNN
+F 0 "#PWR8" H 4400 2850 50  0001 C CNN
 F 1 "VCC" H 4400 3150 50  0000 C CNN
 F 2 "" H 4400 3000 50  0000 C CNN
@@
 Wire Wire Line
 	4500 6900 4500 8600
-Wire Wire Line
-	9800 8800 10200 8800
-Wire Wire Line
-	10200 8800 10200 8300
-Wire Wire Line
-	10200 8300 10400 8300
-Wire Wire Line
-	10400 7900 10100 7900
-Wire Wire Line
-	10100 7900 10100 8500
-Wire Wire Line
-	10100 8500 9800 8500
 Wire Bus Line
 	700  7200 9900 7200
@@
 Wire Bus Line
 	13650 2250 13650 3250
+$Sheet
+S 12400 4400 900  1000
+U 5696E359
+F0 "Video Encoder" 60
+F1 "VideoEncoder.sch" 60
+F2 "R" I L 12400 4750 60
+F3 "G" I L 12400 4850 60
+F4 "B" I L 12400 4950 60
+F5 "AUDIO" I L 12400 5250 60
+F6 "NTSC/PAL" O L 12400 5150 60
+F7 "CSYNC" I L 12400 5050 60
+F8 "VIDEO_CLK" I L 12400 4550 60
+$EndSheet
+NoConn ~ 11900 5700
+NoConn ~ 11900 5800
+Wire Wire Line
+	11900 5900 11950 5900
+Wire Wire Line
+	11950 5900 11950 4750
+Wire Wire Line
+	11950 4750 12400 4750
+Wire Wire Line
+	11900 6000 12000 6000
+Wire Wire Line
+	12000 6000 12000 4850
+Wire Wire Line
+	12000 4850 12400 4850
+Wire Wire Line
+	11900 6100 12050 6100
+Wire Wire Line
+	12050 6100 12050 4950
+Wire Wire Line
+	12050 4950 12400 4950
+NoConn ~ 11900 6300
+Wire Wire Line
+	11900 6500 12200 6500
+Wire Wire Line
+	11900 6200 12100 6200
+Wire Wire Line
+	12100 6200 12100 5050
+Wire Wire Line
+	12100 5050 12400 5050
+Wire Wire Line
+	11900 6400 12150 6400
+Wire Wire Line
+	12150 6400 12150 5150
+Wire Wire Line
+	12150 5150 12400 5150
+Wire Wire Line
+	12200 6500 12200 5250
+Wire Wire Line
+	12200 5250 12400 5250
+$Sheet
+S 10700 4050 700  700
+U 56974E9D
+F0 "Clock Generation" 60
+F1 "ClockGen.sch" 60
+F2 "VIDEO_CLK" O R 11400 4550 60
+F3 "VDP_CLK" O R 11400 4650 60
+$EndSheet
+Wire Wire Line
+	11400 4550 12400 4550
+Wire Wire Line
+	11400 4650 11800 4650
+Text Label 11800 4650 2    60   ~ 0
+VDP_CLK
+Text Label 10050 8500 0    60   ~ 0
+VDP_CLK
+Wire Wire Line
+	10050 8500 10400 8500
 $EndSCHEMATC

Commit message: A bit more video circuitry
Connections:
- net CONT: now reaches CN2.34 (CONT), CN3.34 (CONT), CN4.34 (CONT)
Changed lines of the file:
@@
 	4000 1300 4000 3300
 Wire Wire Line
-	4100 1300 4100 3000
+	4100 1300 4100 3700
 Wire Wire Line
 	4200 1300 4200 3100
@@
 Wire Wire Line
 	10050 8500 10400 8500
+Text Label 4100 3700 1    60   ~ 0
+CONT
+Connection ~ 4100 3000
 $EndSCHEMATC

Commit message: Main digital sections should now be complete
Parts:
- added C?: 10uF, Capacitors_ThroughHole:C_Disc_D3_P2.5, symbol C_Small
- added D?: D_Small, symbol D_Small
- added R?: 100K, Resistors_ThroughHole:Resistor_Horizontal_RM10mm, symbol R_Small
Connections:
- net A15: now also CN3.36 (A15), CN4.36 (A15)
- net BUSAK: now also CN3.45 (BusAck), CN4.45 (BusAck)
- net BUSRQ: now also CN3.44 (BusReq), CN4.44 (BusReq)
- net CONT: now also IC4.42 (#CONT1)
- net EXM1: now also IC3.16 (#EXM1)
- net EXM2: now also IC1.22 (#OE), IC3.17 (#EXM2)
- net GNDPWR: now also C?.1
- net HALT: now also CN3.40 (Halt), CN4.40 (Halt)
- net INT: now also CN3.42 (Int)
- net KILLGA: now also CN3.43 (KILLGA)
- net M1: now also CN3.37 (M1), CN4.37 (M1)
- net NMI: now also CN3.50 (NMI), CN4.50 (NMI)
- net VCC: now also D?.1 (K), R?.1
- net WAIT: now also CN3.41 (Wait), CN4.41 (Wait)
- net #RESET: now reaches U2.26 (#RESET)
- net #RESET: now also CN3.46 (Reset), CN4.46 (Reset), IC3.23 (#RESET), IC4.41 (#RST), C?.2, D?.2 (A), R?.2
- net CLK: now reaches U2.6 (CLK)
- net CLK: now also CN3.47 (Clock), CN4.47 (Clock), IC3.34 (CLK)
- net CSRAM: now reaches IC4.24 (#CSRAM)
- net CSRAM: now also CN3.49 (CSRAM), CN4.49 (CSRAM), IC3.15 (#CSRAM)
- net at IC4.33 (#H-L): now also IC3.35 (#H-L)
- net KBSEL: now reaches IC3.14 (#KBSEL)
- net KBSEL: now also CN3.48 (KBSEL), CN4.48 (KBSEL)
- net IOREQ: now reaches CN3.38 (IOReq), CN4.38 (IOReq)
- net REFSH: now reaches CN3.39 (Refresh), CN4.39 (Refresh)
- net at CN4.42 (Int): no longer CN3.42 (Int)
- net at CN4.43 (KILLGA): no longer CN3.43 (KILLGA)
Other:
- note added: "CPU"
- note added: "Reset"
