File: VideoEncoder.sch (KiCad schematic (older format))
At the start: 17 parts, among them IC9 CXA1145P, P1 DIN_8

Commit message: A bit more video circuitry
Parts:
- added C?: 180pF, symbol CP_Small
- added C? (x2): 12pF, symbol C_Small
- added C?: 100nF, symbol C_Small
- added C?: 10nF, symbol C_Small
- added C?: 100p, symbol CP_Small
- added C?: 470uF, symbol C_Small
- added IC10: 74HC132, symbol 74LS132
- added L? (x2): 100uH, symbol INDUCTOR_SMALL
- added L?: 12uH, symbol INDUCTOR_SMALL
- added R?: 2.2K, Resistors_ThroughHole:Resistor_Horizontal_RM10mm, symbol R_Small
- added R? (x2): 1K, Resistors_ThroughHole:Resistor_Horizontal_RM10mm, symbol R_Small
- added R? (x2): 10K, Resistors_ThroughHole:Resistor_Horizontal_RM10mm, symbol R_Small
Connections:
- net GNDPWR: now also IC9.7 (NTSC/PAL), C?.2, C?.2, C?.2, L?.2, R?.2, R?.2
- net VCC: now also IC10.14 (VCC), IC10.14 (VCC), IC10.14 (VCC), IC10.14 (VCC)
- net at IC9.10 (C-SYNCin): now also IC10.8
- net at IC9.12 (VCC): now also IC10.1
- net at IC9.14 (Vref): now also IC9.18 (Yin), C?.1, C?.1, C?.2, L?.1
- net at IC9.15 (CHROMAout): now also R?.2
- net at IC9.16 (Yout): now also R?.1
- net at IC9.17 (CHROMAin): now also C?.2
- net at IC9.21 (Bout): now also P1.7 (_); no longer P1.8
- net at IC9.22 (Gout): now also P1.8; no longer P1.4
- net at IC9.23 (Rout): now also P1.4; no longer P1.7 (_)
- new net: C?.1, L?.2, R?.2
- new net: C?.1, L?.1, R?.1
- new net: C?.2, L?.2
- new net: C?.1, C?.1, L?.1, R?.1
- new net: IC10.10, IC10.11
- new net: IC10.6, IC10.9
- new net: IC10.13, IC10.4
- new net: C?.1, IC10.5, R?.1
- new net: IC10.12, R?.2
- new net: IC10.2, R?.1
- new net: C?.2, IC10.3
- new net GND: IC10.7 (GND), IC10.7 (GND), IC10.7 (GND), IC10.7 (GND)
- no-connect marks 1 -> 2
Other:
- moved on the sheet: C14, C15, P1
